File: Voyager97.kicad_pcb (KiCad board)
At the start: 2 copper layers, 388.9 x 122.2 mm, 354 parts, among them J1 AVR-ISP-6, Q1 DSS60601MZ4-13, U1 AT90USB1286-AU, U2 PRTR5V0U2X, Y1 16MHz

Commit message: Update to new universal logo
Parts:
- added G***: LOGO, locallib:ai-outline-7.6, F.Cu at (384.2, 109.5)
- added SW1: SW_Push, Molex-0548190589:SKQG-1155865, B.Cu at (403.2, 47.6)
- moved G*** 3.97 mm to (135.7, 136.5) (x2)
Routing:
- net RESET: track 41.3 -> 76.6 mm
- net GND: track 199.0 -> 215.1 mm
- net LEDGND: track 2344.7 -> 2344.3 mm, vias 16 -> 17
Other:
- net class Power: trace_width 0.635 -> 0.381
- board text added: "Voyager97 PCB Rev 1.2"
- board text added: "kb.ai03.me"
- board text removed: "Compact Fullsize Keyboard PCB by ai03"
- board text removed: "Designed by ai03"
