File: Voyager97.sch (KiCad schematic (older format))
At the start: 22 parts, among them J1 AVR-ISP-6, Q1 DSS60601MZ4-13, SW1 SW_Push, U1 AT90USB1286-AU, U2 PRTR5V0U2X, Y1 16MHz

Commit message: Add more flex cutouts
Parts:
- removed SW1: SW_Push, Molex-0548190589:PushButton_6x6mm_TH, symbol Switch:SW_Push
Connections:
- wire segments 84 -> 82
Changed lines of the file:
@@
-	1    0    0    -1
-$EndComp
-$Comp
-L Switch:SW_Push SW1
-U 1 1 5B32EDAB
-P 2900 3275
-F 0 "SW1" H 2950 3375 50  0000 L CNN
-F 1 "SW_Push" H 2900 3215 50  0000 C CNN
-F 2 "Molex-0548190589:PushButton_6x6mm_TH" H 2900 3475 50  0001 C CNN
-F 3 "" H 2900 3475 50  0001 C CNN
-	1    2900 3275
-	1    0    0    -1
-$EndComp
-$Comp
-L power:GND #PWR06
-U 1 1 5B32EDDE
-P 2700 3350
-F 0 "#PWR06" H 2700 3100 50  0001 C CNN
-F 1 "GND" H 2700 3200 50  0000 C CNN
-F 2 "" H 2700 3350 50  0001 C CNN
-F 3 "" H 2700 3350 50  0001 C CNN
-	1    2700 3350
 	1    0    0    -1
 $EndComp
@@
 	5975 4875 6225 4875
 Wire Wire Line
-	3100 3275 3300 3275
-Connection ~ 3300 3275
-Wire Wire Line
-	2700 3350 2700 3275
-Wire Wire Line
 	3525 4575 3925 4575

Commit message: Update to new universal logo
Parts:
- added SW1: SW_Push, Molex-0548190589:SKQG-1155865, symbol Switch:SW_Push
Connections:
- wire segments 82 -> 84
Changed lines of the file:
@@
 	1550 2475 1700 2475
 NoConn ~ 3925 3875
+$Comp
+L Switch:SW_Push SW1
+U 1 1 5C4DB62B
+P 2975 3275
+F 0 "SW1" H 2975 3560 50  0000 C CNN
+F 1 "SW_Push" H 2975 3469 50  0000 C CNN
+F 2 "Molex-0548190589:SKQG-1155865" H 2975 3475 50  0001 C CNN
+F 3 "" H 2975 3475 50  0001 C CNN
+	1    2975 3275
+	1    0    0    -1
+$EndComp
+Wire Wire Line
+	3175 3275 3300 3275
+Connection ~ 3300 3275
+Wire Wire Line
+	2775 3275 2575 3275
+$Comp
+L power:GND #PWR?
+U 1 1 5C4DF5AA
+P 2575 3275
+F 0 "#PWR?" H 2575 3025 50  0001 C CNN
+F 1 "GND" H 2580 3102 50  0000 C CNN
+F 2 "" H 2575 3275 50  0001 C CNN
+F 3 "" H 2575 3275 50  0001 C CNN
+	1    2575 3275
+	1    0    0    -1
+$EndComp
 $EndSCHEMATC
